Commit message: add lidar to the simulation

File: src/apricotka-robot-car/description/robot.urdf.xacro (robot description, xacro)
@@ -10,3 +10,4 @@
     <xacro:include filename="ros2_control.xacro" />
     <xacro:include filename="imu.xacro" />
+    <xacro:include filename="lidar.xacro" />
 </robot>

File: src/apricotka-robot-car/description/water_tank.xacro (robot description, xacro)
@@ -6,5 +6,5 @@
     <xacro:property name="tank_mass" value="100" />
     <xacro:property name="cap_radius" value="0.1" />
-    <xacro:property name="cap_height" value="0.05" />
+    <xacro:property name="cap_height" value="0.025" />
     <link name="water_tank_link">
         <visual>
