Commit message: add slam_toolbox mapping & localization

File: src/apricotka-robot-car/description/lidar.xacro (robot description, xacro)
@@ -4,5 +4,5 @@
         <parent link="water_tank_link"/>
         <child link="laser_frame"/>
-        <origin xyz="0 0 0.15" rpy="0 0 0"/>
+        <origin xyz="0 0 0.08" rpy="0 0 0"/>
     </joint>
     <link name="laser_frame">

File: src/apricotka-robot-car/description/robot.urdf.xacro (robot description, xacro)
@@ -7,5 +7,5 @@
     <xacro:include filename="camera.xacro" />
     <xacro:include filename="water_tank.xacro" />
-    <xacro:include filename="flexible_rod.xacro" />
+<!--<xacro:include filename="flexible_rod.xacro" />-->
     <xacro:include filename="ros2_control.xacro" />
     <xacro:include filename="imu.xacro" />

File: src/apricotka-robot-car/description/robot_core.xacro (robot description, xacro)
@@ -21,7 +21,7 @@
     </link>
     <joint name="base_footprint_joint" type="fixed">
-        <parent link="base_link"/>
-        <child link="base_footprint"/>
-        <origin xyz="0 0 0" rpy="0 0 0"/>
+        <origin xyz="0 0 ${wheel_radius}" rpy="0 0 0" />
+        <parent link="base_footprint"/>
+        <child link="base_link" />
     </joint>
     <!-- chassis -->

File: src/apricotka-robot-car/description/water_tank.xacro (robot description, xacro)
@@ -3,5 +3,5 @@
     <xacro:property name="tank_x_size" value="0.6" />
     <xacro:property name="tank_y_size" value="0.6" />
-    <xacro:property name="tank_z_size" value="0.32" />
+    <xacro:property name="tank_z_size" value="0.25" />
     <xacro:property name="tank_mass" value="100" />
     <xacro:property name="cap_radius" value="0.1" />
