Commit message: Issue #11: Change robot appearance

File: description/robot.urdf.xacro (robot description, xacro)
@@ -1,7 +1,11 @@
 <?xml version="1.0"?>
 <robot xmlns:xacro="http://www.ros.org/wiki/xacro"  name="robot">
-    <xacro:arg name="sim_mode" default="false"/>
+    <xacro:arg name="sim_mode" default="true"/>
+    <xacro:include filename="materials.xacro" />
+    <xacro:include filename="inertia.xacro" />
     <xacro:include filename="robot_core.xacro" />
     <xacro:include filename="camera.xacro" />
+    <xacro:include filename="water_tank.xacro" />
+<!-- <xacro:include filename="flexible_rod.xacro" /> -->
     <xacro:include filename="ros2_control.xacro" />
 </robot>

File: description/robot_core.xacro (robot description, xacro)
@@ -1,56 +1,17 @@
 <?xml version="1.0"?>
 <robot xmlns:xacro="http://www.ros.org/wiki/xacro" >
-    <!-- define colors -->
-    <material name="white">
-        <color rgba="1 1 1 1" />
-    </material>
-    <material name="blue">
-        <color rgba="${0/255} ${0/255} ${255/255} 1.0"/>
-    </material>
-    <!-- define gazebo materials -->
-    <material name="gazebo_white">
-        <color rgba="1 1 1 1" />
-        <ambient>1 1 1 1</ambient>
-        <diffuse>1 1 1 1</diffuse>
-        <specular>.1 .1 .1 128</specular>
-    </material>
-    <material name="gazebo_blue">
-        <color rgba="${0/255} ${0/255} ${255/255} 1.0"/>
-        <ambient>0 0 1</ambient>
-        <diffuse>0 0 1</diffuse>
-        <specular>0.1 0.1 0.1 1 1</specular>
-    </material>
     <!-- base dimensions -->
-    <xacro:property name="base_x_size" value="0.25" />
-    <xacro:property name="base_y_size" value="0.1" />
-    <xacro:property name="base_z_size" value="0.035" />
+    <xacro:property name="base_x_size" value="1.0" />
+    <xacro:property name="base_y_size" value="0.65" />
+    <xacro:property name="base_z_size" value="0.1" />
     <!-- wheel properties -->
-    <xacro:property name="wheel_length" value="0.025" />
-    <xacro:property name="wheel_radius" value="0.033" />
+    <xacro:property name="wheel_length" value="0.114" />
+    <xacro:property name="wheel_radius" value="0.183" />
     <!-- material density -->
     <xacro:property name="base_density" value="1500.0" />
-    <xacro:property name="wheel_density" value="1500.0" />
+    <xacro:property name="wheel_density" value="400.0" />
     <!-- base and wheel mass -->
     <xacro:property name="base_mass" value="${base_density*base_x_size*base_y_size*base_z_size}" />
     <xacro:property name="wheel_mass" value="${wheel_density*pi*wheel_radius*wheel_radius*wheel_length}" />
-    <!-- Inertia macro -->
-    <xacro:macro name="inertial_box" params="mass x y z *origin">
-        <inertial>
-            <xacro:insert_block name="origin"/>
-            <mass value="${mass}" />
-            <inertia ixx="${(1/12) * mass * (y*y+z*z)}" ixy="0.0" ixz="0.0"
-                    iyy="${(1/12) * mass * (x*x+z*z)}" iyz="0.0"
-                    izz="${(1/12) * mass * (x*x+y*y)}" />
-        </inertial>
-    </xacro:macro>
-    <xacro:macro name="inertial_cylinder" params="mass length radius *origin">
-        <inertial>
-            <xacro:insert_block name="origin"/>
-            <mass value="${mass}" />
-            <inertia ixx="${(1/12) * mass * (3*radius*radius + length*length)}" ixy="0.0" ixz="0.0"
-                    iyy="${(1/12) * mass * (3*radius*radius + length*length)}" iyz="0.0"
-                    izz="${(1/2) * mass * (radius*radius)}" />
-        </inertial>
-    </xacro:macro>
     <!-- base link -->
     <link name="base_link">
@@ -115,10 +76,6 @@
         <gazebo reference="${prefix}_link">
             <material name="gazebo_blue"/>
-            <!-- <xacro:if value="${x_reflect == 1}">
-                <mu1 value="0.001"/>
-                <mu2 value="0.001"/>
-            </xacro:if> -->
-            <mu1 value="5"/>
-            <mu2 value="5"/>
+            <!-- <mu1 value="5"/>
+            <mu2 value="5"/> -->
         </gazebo>
     </xacro:macro>

File: description/ros2_control.xacro (robot description, xacro)
@@ -15,14 +15,18 @@
             <hardware>
                 <plugin>diffdrive_arduino/DiffDriveArduinoHardware</plugin>
-                <param name="left_wheel_name">front_left_wheel_joint</param>
-                <param name="right_wheel_name">front_right_wheel_joint</param>
+                <param name="left_wheel_name">rear_left_wheel_joint</param>
+                <param name="right_wheel_name">rear_right_wheel_joint</param>
                 <param name="loop_rate">30</param>
                 <param name="device">/dev/ttyUSB0</param>
                 <param name="baud_rate">115200</param>
                 <param name="timeout_ms">1000</param>
-                <param name="enc_counts_per_rev">3436</param>
+                <param name="enc_counts_per_rev">41</param>
+                <param name="pid_p">20</param>
+                <param name="pid_d">12</param>
+                <param name="pid_i">0</param>
+                <param name="pid_o">50</param>
             </hardware>
-            <xacro:wheel_interface prefix="front_left_wheel" />
-            <xacro:wheel_interface prefix="front_right_wheel" />
+            <!-- <xacro:wheel_interface prefix="front_left_wheel" />
+            <xacro:wheel_interface prefix="front_right_wheel" /> -->
             <xacro:wheel_interface prefix="rear_left_wheel" />
             <xacro:wheel_interface prefix="rear_right_wheel" />
@@ -45,4 +49,4 @@
           <parameters>$(find apricotka-robot-car)/config/my_controllers.yaml</parameters>
         </plugin>
-      </gazebo>
+    </gazebo>
 </robot>
