Commit message: Issue #12: Implement ros2_control hardware interface for IMU

File: description/ros2_control.xacro (robot description, xacro)
@@ -25,4 +25,23 @@
         </ros2_control>
     </xacro:unless>
+    <xacro:unless value="$(arg sim_mode)">
+        <ros2_control name="KPIRoverIMUHW" type="sensor">
+            <hardware>
+                <plugin>kpi_rover_imu_hw/KPIRoverIMUHW</plugin>
+                <param name="udp_port">$(arg udp_port)</param>
+            </hardware>
+            <joint name="imu_joint">
+                <state_interface name="orientation.x" />
+                <state_interface name="orientation.y" />
+                <state_interface name="orientation.z" />
+                <state_interface name="angular_velocity.x" />
+                <state_interface name="angular_velocity.y" />
+                <state_interface name="angular_velocity.z" />
+                <state_interface name="linear_acceleration.x" />
+                <state_interface name="linear_acceleration.y" />
+                <state_interface name="linear_acceleration.z" />
+            </joint>
+        </ros2_control>
+    </xacro:unless>
     <xacro:if value="$(arg sim_mode)">
         <ros2_control name="GazeboSystem" type="system">
