Commit message: Issue #30: Change robot collor

File: description/materials.xacro (robot description, xacro)
@@ -4,4 +4,7 @@
     <material name="white">
         <color rgba="1 1 1 1" />
+    </material>
+    <material name="yellow">
+        <color rgba="1 1 0 1"/>
     </material>
     <material name="blue">

File: description/robot_core.xacro (robot description, xacro)
@@ -33,5 +33,5 @@
                 <mesh filename = "package://kpi_rover/description/meshes/kpi_rover_body.stl" scale="0.001 0.001 0.001"/>
             </geometry>
-            <material name="white"/>
+            <material name="yellow"/>
         </visual>
         <collision>
