Commit message: Issue #30: Add IMU link

File: description/imu.xacro (robot description, xacro)
@@ -4,5 +4,5 @@
         <parent link="base_link"/>
         <child link="imu_link"/>
-        <origin xyz="0.0 0 0.068" rpy="0 0 0"/>
+        <origin xyz="-0.036 0.039 0.015" rpy="0 0 0"/>
     </joint>
     <link name="imu_link"/>

File: description/robot.urdf.xacro (robot description, xacro)
@@ -10,5 +10,5 @@
     <!-- <xacro:include filename="flexible_rod.xacro" /> -->
     <xacro:include filename="ros2_control.xacro" />
-    <!-- <xacro:include filename="imu.xacro" /> -->
+    <xacro:include filename="imu.xacro" />
     <xacro:include filename="lidar.xacro" />
 </robot>

Commit message: Issue #30: Add IMU link

File: description/imu.xacro (robot description, xacro)
@@ -4,5 +4,5 @@
         <parent link="base_link"/>
         <child link="imu_link"/>
-        <origin xyz="0.0 0 0.068" rpy="0 0 0"/>
+        <origin xyz="-0.036 0.039 0.015" rpy="0 0 0"/>
     </joint>
     <link name="imu_link"/>
