Commit message: Issue #11: Fixed odometry drift caused by ros2_control

File: description/robot_core.xacro (robot description, xacro)
@@ -21,7 +21,7 @@
     </link>
     <joint name="base_footprint_joint" type="fixed">
-        <parent link="base_link"/>
-        <child link="base_footprint"/>
-        <origin xyz="0 0 0" rpy="0 0 0"/>
+        <parent link="base_footprint"/>
+        <child link="base_link"/>
+        <origin xyz="0 0 ${wheel_radius}" rpy="0 0 0"/>
     </joint>
     <!-- chassis -->
@@ -51,5 +51,5 @@
     </gazebo>
     <!-- wheels -->
-    <xacro:macro name="wheel" params="prefix x_reflect y_reflect">
+    <xacro:macro name="wheel" params="prefix x_reflect y_reflect mu1 mu2">
         <link name="${prefix}_link">
             <visual>
@@ -76,11 +76,11 @@
         <gazebo reference="${prefix}_link">
             <material name="gazebo_blue"/>
-            <!-- <mu1 value="5"/>
-            <mu2 value="5"/> -->
+            <mu1 value="${mu1}"/>
+ <!--           <mu2 value="${mu2}"/> -->
         </gazebo>
     </xacro:macro>
-    <xacro:wheel prefix="front_left_wheel" x_reflect="1" y_reflect="1" />
-    <xacro:wheel prefix="front_right_wheel" x_reflect="1" y_reflect="-1" />
-    <xacro:wheel prefix="rear_left_wheel" x_reflect="-1" y_reflect="1" />
-    <xacro:wheel prefix="rear_right_wheel" x_reflect="-1" y_reflect="-1" />
+    <xacro:wheel prefix="front_left_wheel" x_reflect="1" y_reflect="1" mu1="0.0" mu2="0.0"/>
+    <xacro:wheel prefix="front_right_wheel" x_reflect="1" y_reflect="-1" mu1="0.0" mu2="0.0"/>
+    <xacro:wheel prefix="rear_left_wheel" x_reflect="-1" y_reflect="1" mu1="5.0" mu2="0.2"/>
+    <xacro:wheel prefix="rear_right_wheel" x_reflect="-1" y_reflect="-1" mu1="5.0" mu2="0.2"/>
 </robot>

Commit message: Issue #30: Change robot collor

File: description/robot_core.xacro (robot description, xacro)
@@ -33,5 +33,5 @@
                 <mesh filename = "package://kpi_rover/description/meshes/kpi_rover_body.stl" scale="0.001 0.001 0.001"/>
             </geometry>
-            <material name="white"/>
+            <material name="yellow"/>
         </visual>
         <collision>

Commit message: Change robot size parameters according to the real one

File: description/robot_core.xacro (robot description, xacro)
@@ -2,10 +2,10 @@
 <robot xmlns:xacro="http://www.ros.org/wiki/xacro" >
     <!-- base dimensions -->
-    <xacro:property name="base_x_size" value="1.0" />
-    <xacro:property name="base_y_size" value="0.65" />
-    <xacro:property name="base_z_size" value="0.1" />
+    <xacro:property name="base_x_size" value="0.24" />
+    <xacro:property name="base_y_size" value="0.18" />
+    <xacro:property name="base_z_size" value="0.01" />
     <!-- wheel properties -->
-    <xacro:property name="wheel_length" value="0.114" />
-    <xacro:property name="wheel_radius" value="0.183" />
+    <xacro:property name="wheel_length" value="0.04" />
+    <xacro:property name="wheel_radius" value="0.04" />
     <!-- material density -->
     <xacro:property name="base_density" value="1500.0" />

File: description/water_tank.xacro (robot description, xacro)
@@ -1,10 +1,10 @@
 <?xml version="1.0"?>
 <robot xmlns:xacro="http://www.ros.org/wiki/xacro">
-    <xacro:property name="tank_x_size" value="0.6" />
-    <xacro:property name="tank_y_size" value="0.6" />
-    <xacro:property name="tank_z_size" value="0.32" />
-    <xacro:property name="tank_mass" value="100" />
-    <xacro:property name="cap_radius" value="0.1" />
-    <xacro:property name="cap_height" value="0.025" />
+    <xacro:property name="tank_x_size" value="0.15" />
+    <xacro:property name="tank_y_size" value="0.15" />
+    <xacro:property name="tank_z_size" value="0.1" />
+    <xacro:property name="tank_mass" value="1" />
+    <xacro:property name="cap_radius" value="0.01" />
+    <xacro:property name="cap_height" value="0.0025" />
     <link name="water_tank_link">
         <visual>

Commit message: Issue #28: Change robot size parameters according to the real one

File: description/robot_core.xacro (robot description, xacro)
@@ -2,10 +2,10 @@
 <robot xmlns:xacro="http://www.ros.org/wiki/xacro" >
     <!-- base dimensions -->
-    <xacro:property name="base_x_size" value="1.0" />
-    <xacro:property name="base_y_size" value="0.65" />
-    <xacro:property name="base_z_size" value="0.1" />
+    <xacro:property name="base_x_size" value="0.24" />
+    <xacro:property name="base_y_size" value="0.18" />
+    <xacro:property name="base_z_size" value="0.01" />
     <!-- wheel properties -->
-    <xacro:property name="wheel_length" value="0.114" />
-    <xacro:property name="wheel_radius" value="0.183" />
+    <xacro:property name="wheel_length" value="0.04" />
+    <xacro:property name="wheel_radius" value="0.04" />
     <!-- material density -->
     <xacro:property name="base_density" value="1500.0" />

File: description/water_tank.xacro (robot description, xacro)
@@ -5,6 +5,6 @@
     <xacro:property name="tank_z_size" value="0.32" />
     <xacro:property name="tank_mass" value="100" />
-    <xacro:property name="cap_radius" value="0.1" />
-    <xacro:property name="cap_height" value="0.025" />
+    <xacro:property name="cap_radius" value="0.01" />
+    <xacro:property name="cap_height" value="0.0025" />
     <link name="water_tank_link">
         <visual>
