Commit message: Issue #30: Fix URDF

File: description/lidar.xacro (robot description, xacro)
@@ -2,13 +2,12 @@
 <robot xmlns:xacro="http://www.ros.org/wiki/xacro" >
     <joint name="laser_joint" type="fixed">
-        <parent link="water_tank_link"/>
+        <parent link="base_link"/>
         <child link="laser_frame"/>
-        <origin xyz="0 0 0.15" rpy="0 0 0"/>
+        <origin xyz="0 0 0.11" rpy="0 0 0"/>
     </joint>
     <link name="laser_frame">
         <visual>
-            <origin xyz="0.1 0 0.05" rpy="0 0 0"/>
             <geometry>
-                <mesh filename = "package://description/meshes/lidar.dae"/>
+                <mesh filename = "package://kpi_rover/description/meshes/lidar.stl" scale="0.001 0.001 0.001"/>
             </geometry>
         </visual>

File: description/robot_core.xacro (robot description, xacro)
@@ -2,10 +2,12 @@
 <robot xmlns:xacro="http://www.ros.org/wiki/xacro" >
     <!-- base dimensions -->
-    <xacro:property name="base_x_size" value="1.0" />
-    <xacro:property name="base_y_size" value="0.65" />
+    <xacro:property name="base_x_size" value="0.21" />
+    <xacro:property name="base_y_size" value="0.15" />
     <xacro:property name="base_z_size" value="0.1" />
     <!-- wheel properties -->
-    <xacro:property name="wheel_length" value="0.114" />
-    <xacro:property name="wheel_radius" value="0.183" />
+    <xacro:property name="wheel_radius" value="0.035" />
+    <xacro:property name="axle_separation" value="0.140" />
+    <xacro:property name="wheel_separation" value="0.220" />
+    <xacro:property name="axis_offset_from_base" value="0.035" />
     <!-- material density -->
     <xacro:property name="base_density" value="1500.0" />
@@ -13,5 +15,5 @@
     <!-- base and wheel mass -->
     <xacro:property name="base_mass" value="${base_density*base_x_size*base_y_size*base_z_size}" />
-    <xacro:property name="wheel_mass" value="${wheel_density*pi*wheel_radius*wheel_radius*wheel_length}" />
+    <xacro:property name="wheel_mass" value="${wheel_density*pi*wheel_radius*wheel_radius*0.020}" />
     <!-- base link -->
     <link name="base_link">
@@ -28,13 +30,13 @@
     <link name="chassis">
         <visual>
-        <geometry>
-            <box size="${base_x_size} ${base_y_size} ${base_z_size}"/>
-        </geometry>
-        <material name="white"/>
+            <geometry>
+                <mesh filename = "package://kpi_rover/description/meshes/kpi_rover_body.stl" scale="0.001 0.001 0.001"/>
+            </geometry>
+            <material name="white"/>
         </visual>
         <collision>
-        <geometry>
-            <box size="${base_x_size} ${base_y_size} ${base_z_size}"/>
-        </geometry>
+            <geometry>
+                <mesh filename = "package://kpi_rover/description/meshes/kpi_rover_body.stl" scale="0.001 0.001 0.001"/>
+            </geometry>
         </collision>
         <xacro:inertial_box mass="${base_mass}" x="${base_x_size}" y="${base_y_size}" z="${base_z_size}">
@@ -55,5 +57,5 @@
             <visual>
                 <geometry>
-                    <cylinder length="${wheel_length}" radius="${wheel_radius}" />
+                    <mesh filename = "package://kpi_rover/description/meshes/wheel.stl" scale="0.001 0.001 0.001"/>
                 </geometry>
                 <material name="blue"/>
@@ -61,16 +63,16 @@
             <collision>
                 <geometry>
-                    <sphere radius="${wheel_radius}" />
+                    <mesh filename = "package://kpi_rover/description/meshes/wheel.stl" scale="0.001 0.001 0.001"/>
                 </geometry>
             </collision>
-            <xacro:inertial_cylinder mass="${wheel_mass}" length="${wheel_length}" radius="${wheel_radius}">
+            <xacro:inertial_cylinder mass="${wheel_mass}" length="0.020" radius="${wheel_radius}">
                 <origin xyz="0 0 0" rpy="0 0 0"/>
             </xacro:inertial_cylinder>
         </link>
-        <joint name="${prefix}_joint" type="continuous">
+        <joint name="${prefix}_joint" type="fixed">
             <parent link="base_link"/>
             <child link="${prefix}_link"/>
-            <origin xyz="${x_reflect*(base_x_size/4)} ${y_reflect*(base_y_size + wheel_length)/2} 0" rpy="${-1*y_reflect*pi/2} 0 0"/>
-            <axis xyz="0 0 ${y_reflect}"/>
+            <origin xyz="${x_reflect*axle_separation/2} ${y_reflect*wheel_separation/2} ${-axis_offset_from_base}" rpy="${-y_reflect*pi/2} 0 0"/>
+            <axis xyz="0 0 0"/>
         </joint>
         <gazebo reference="${prefix}_link">

Commit message: Issue #30: Fix URDF

File: description/lidar.xacro (robot description, xacro)
@@ -2,13 +2,12 @@
 <robot xmlns:xacro="http://www.ros.org/wiki/xacro" >
     <joint name="laser_joint" type="fixed">
-        <parent link="water_tank_link"/>
+        <parent link="base_link"/>
         <child link="laser_frame"/>
-        <origin xyz="0 0 0.15" rpy="0 0 0"/>
+        <origin xyz="0 0 0.11" rpy="0 0 0"/>
     </joint>
     <link name="laser_frame">
         <visual>
-            <origin xyz="0.1 0 0.05" rpy="0 0 0"/>
             <geometry>
-                <mesh filename = "package://description/meshes/lidar.dae"/>
+                <mesh filename = "package://kpi_rover/description/meshes/lidar.stl" scale="0.001 0.001 0.001"/>
             </geometry>
         </visual>

File: description/robot.urdf.xacro (robot description, xacro)
@@ -7,9 +7,8 @@
     <xacro:include filename="inertia.xacro" />
     <xacro:include filename="robot_core.xacro" />
-    <xacro:include filename="camera.xacro" />
-    <xacro:include filename="water_tank.xacro" />
-<!-- <xacro:include filename="flexible_rod.xacro" /> -->
+    <!-- <xacro:include filename="camera.xacro" /> -->
+    <!-- <xacro:include filename="flexible_rod.xacro" /> -->
     <xacro:include filename="ros2_control.xacro" />
-    <xacro:include filename="imu.xacro" />
+    <!-- <xacro:include filename="imu.xacro" /> -->
     <xacro:include filename="lidar.xacro" />
 </robot>

File: description/robot_core.xacro (robot description, xacro)
@@ -2,10 +2,12 @@
 <robot xmlns:xacro="http://www.ros.org/wiki/xacro" >
     <!-- base dimensions -->
-    <xacro:property name="base_x_size" value="1.0" />
-    <xacro:property name="base_y_size" value="0.65" />
+    <xacro:property name="base_x_size" value="0.21" />
+    <xacro:property name="base_y_size" value="0.15" />
     <xacro:property name="base_z_size" value="0.1" />
     <!-- wheel properties -->
-    <xacro:property name="wheel_length" value="0.114" />
-    <xacro:property name="wheel_radius" value="0.183" />
+    <xacro:property name="wheel_radius" value="0.035" />
+    <xacro:property name="axle_separation" value="0.140" />
+    <xacro:property name="wheel_separation" value="0.220" />
+    <xacro:property name="axis_offset_from_base" value="0.035" />
     <!-- material density -->
     <xacro:property name="base_density" value="1500.0" />
@@ -13,5 +15,5 @@
     <!-- base and wheel mass -->
     <xacro:property name="base_mass" value="${base_density*base_x_size*base_y_size*base_z_size}" />
-    <xacro:property name="wheel_mass" value="${wheel_density*pi*wheel_radius*wheel_radius*wheel_length}" />
+    <xacro:property name="wheel_mass" value="${wheel_density*pi*wheel_radius*wheel_radius*0.020}" />
     <!-- base link -->
     <link name="base_link">
@@ -28,13 +30,13 @@
     <link name="chassis">
         <visual>
-        <geometry>
-            <box size="${base_x_size} ${base_y_size} ${base_z_size}"/>
-        </geometry>
-        <material name="white"/>
+            <geometry>
+                <mesh filename = "package://kpi_rover/description/meshes/kpi_rover_body.stl" scale="0.001 0.001 0.001"/>
+            </geometry>
+            <material name="white"/>
         </visual>
         <collision>
-        <geometry>
-            <box size="${base_x_size} ${base_y_size} ${base_z_size}"/>
-        </geometry>
+            <geometry>
+                <mesh filename = "package://kpi_rover/description/meshes/kpi_rover_body.stl" scale="0.001 0.001 0.001"/>
+            </geometry>
         </collision>
         <xacro:inertial_box mass="${base_mass}" x="${base_x_size}" y="${base_y_size}" z="${base_z_size}">
@@ -55,5 +57,5 @@
             <visual>
                 <geometry>
-                    <cylinder length="${wheel_length}" radius="${wheel_radius}" />
+                    <mesh filename = "package://kpi_rover/description/meshes/wheel.stl" scale="0.001 0.001 0.001"/>
                 </geometry>
                 <material name="blue"/>
@@ -61,16 +63,16 @@
             <collision>
                 <geometry>
-                    <sphere radius="${wheel_radius}" />
+                    <mesh filename = "package://kpi_rover/description/meshes/wheel.stl" scale="0.001 0.001 0.001"/>
                 </geometry>
             </collision>
-            <xacro:inertial_cylinder mass="${wheel_mass}" length="${wheel_length}" radius="${wheel_radius}">
+            <xacro:inertial_cylinder mass="${wheel_mass}" length="0.020" radius="${wheel_radius}">
                 <origin xyz="0 0 0" rpy="0 0 0"/>
             </xacro:inertial_cylinder>
         </link>
-        <joint name="${prefix}_joint" type="continuous">
+        <joint name="${prefix}_joint" type="fixed">
             <parent link="base_link"/>
             <child link="${prefix}_link"/>
-            <origin xyz="${x_reflect*(base_x_size/4)} ${y_reflect*(base_y_size + wheel_length)/2} 0" rpy="${-1*y_reflect*pi/2} 0 0"/>
-            <axis xyz="0 0 ${y_reflect}"/>
+            <origin xyz="${x_reflect*axle_separation/2} ${y_reflect*wheel_separation/2} ${-axis_offset_from_base}" rpy="${-y_reflect*pi/2} 0 0"/>
+            <axis xyz="0 0 0"/>
         </joint>
         <gazebo reference="${prefix}_link">

Commit message: Issue #30: Fix lidar position

File: description/lidar.xacro (robot description, xacro)
@@ -4,5 +4,5 @@
         <parent link="base_link"/>
         <child link="laser_frame"/>
-        <origin xyz="0 0 0.11" rpy="0 0 0"/>
+        <origin xyz="0 0 0.12" rpy="0 0 0"/>
     </joint>
     <link name="laser_frame">
