Commit message: Issue #28: Change robot size parameters according to the real one

File: description/water_tank.xacro (robot description, xacro)
@@ -1,10 +1,10 @@
 <?xml version="1.0"?>
 <robot xmlns:xacro="http://www.ros.org/wiki/xacro">
-    <xacro:property name="tank_x_size" value="0.6" />
-    <xacro:property name="tank_y_size" value="0.6" />
-    <xacro:property name="tank_z_size" value="0.32" />
-    <xacro:property name="tank_mass" value="100" />
-    <xacro:property name="cap_radius" value="0.1" />
-    <xacro:property name="cap_height" value="0.025" />
+    <xacro:property name="tank_x_size" value="0.15" />
+    <xacro:property name="tank_y_size" value="0.15" />
+    <xacro:property name="tank_z_size" value="0.1" />
+    <xacro:property name="tank_mass" value="1.5" />
+    <xacro:property name="cap_radius" value="0.01" />
+    <xacro:property name="cap_height" value="0.0025" />
     <link name="water_tank_link">
         <visual>

Commit message: Fix tank parameters according to real robot

File: description/water_tank.xacro (robot description, xacro)
@@ -1,8 +1,8 @@
 <?xml version="1.0"?>
 <robot xmlns:xacro="http://www.ros.org/wiki/xacro">
-    <xacro:property name="tank_x_size" value="0.6" />
-    <xacro:property name="tank_y_size" value="0.6" />
-    <xacro:property name="tank_z_size" value="0.32" />
-    <xacro:property name="tank_mass" value="100" />
+    <xacro:property name="tank_x_size" value="0.15" />
+    <xacro:property name="tank_y_size" value="0.15" />
+    <xacro:property name="tank_z_size" value="0.1" />
+    <xacro:property name="tank_mass" value="1.5" />
     <xacro:property name="cap_radius" value="0.01" />
     <xacro:property name="cap_height" value="0.0025" />
