Commit message: Issue #43: Change folders structure of kpi_rover_description

File: kpi_rover_description/urdf/lidar.xacro (robot description, xacro)
@@ -10,5 +10,5 @@
             <origin xyz="0.1 0 0.05" rpy="0 0 0"/>
             <geometry>
-                <mesh filename = "package://kpi_rover_description/description/meshes/lidar.dae"/>
+                <mesh filename = "package://kpi_rover_description/meshes/lidar.dae"/>
             </geometry>
         </visual>
