Commit message: Issue #30: Fix wheels positions

File: kpi_rover_description/urdf/imu.xacro (robot description, xacro)
@@ -4,5 +4,5 @@
         <parent link="base_link"/>
         <child link="imu_link"/>
-        <origin xyz="0.0 0 0.068" rpy="0 0 0"/>
+        <origin xyz="0.0 0 0.068" rpy="0 0 -1.57079632679"/>
     </joint>
     <link name="imu_link"/>

File: kpi_rover_description/urdf/lidar.xacro (robot description, xacro)
@@ -4,5 +4,5 @@
         <parent link="water_tank_link"/>
         <child link="laser_frame"/>
-        <origin xyz="0 0 0.15" rpy="0 0 0"/>
+        <origin xyz="0 0 0.15" rpy="0 0 3.14159265359"/>
     </joint>
     <link name="laser_frame">

File: kpi_rover_description/urdf/robot.urdf.xacro (robot description, xacro)
@@ -4,4 +4,5 @@
     <xacro:arg name="serial_device" default="/dev/ttyAMA2"/>
     <xacro:arg name="baud_rate" default="921600"/>
+    <xacro:arg name="encoder_ticks_per_rev" default="1320"/>
     <xacro:include filename="materials.xacro" />
     <xacro:include filename="inertia.xacro" />

File: kpi_rover_description/urdf/ros2_control.xacro (robot description, xacro)
@@ -17,5 +17,5 @@
                 <param name="serial_device">$(arg serial_device)</param>
                 <param name="baud_rate">$(arg baud_rate)</param>
-                <param name="encoder_ticks_per_rev">821</param>
+                <param name="encoder_ticks_per_rev">$(arg encoder_ticks_per_rev)</param>
                 <param name="wheel_radius">0.04</param>
             </hardware>

Commit message: Issue #30: Update URDF

File: kpi_rover_description/urdf/imu.xacro (robot description, xacro)
@@ -4,5 +4,5 @@
         <parent link="base_link"/>
         <child link="imu_link"/>
-        <origin xyz="0.0 0 0.068" rpy="0 0 -1.57079632679"/>
+        <origin xyz="-0.036 0.039 0.015" rpy="0 0 0"/>
     </joint>
     <link name="imu_link"/>
@@ -12,7 +12,4 @@
             <visualize>false</visualize>
             <topic>/imu_broadcaster/imu</topic>
-            <gz_frame_id>imu_link</gz_frame_id>
-            <gaussian_noise>0.01</gaussian_noise>
-            <update_rate>100.0</update_rate>
         </sensor>
     </gazebo>

File: kpi_rover_description/urdf/lidar.xacro (robot description, xacro)
@@ -2,13 +2,12 @@
 <robot xmlns:xacro="http://www.ros.org/wiki/xacro" >
     <joint name="laser_joint" type="fixed">
-        <parent link="water_tank_link"/>
+        <parent link="base_link"/>
         <child link="laser_frame"/>
-        <origin xyz="0 0 0.15" rpy="0 0 3.14159265359"/>
+        <origin xyz="0 0 0.12" rpy="0 0 ${pi}"/>
     </joint>
     <link name="laser_frame">
         <visual>
-            <origin xyz="0.1 0 0.05" rpy="0 0 0"/>
             <geometry>
-                <mesh filename = "package://kpi_rover_description/meshes/lidar.dae"/>
+                <mesh filename = "package://kpi_rover_description/meshes/lidar.stl" scale="0.001 0.001 0.001"/>
             </geometry>
         </visual>

File: kpi_rover_description/urdf/robot.urdf.xacro (robot description, xacro)
@@ -5,10 +5,9 @@
     <xacro:arg name="baud_rate" default="921600"/>
     <xacro:arg name="encoder_ticks_per_rev" default="1320"/>
+    <xacro:arg name="wheel_radius" default="0.034"/>
     <xacro:include filename="materials.xacro" />
     <xacro:include filename="inertia.xacro" />
     <xacro:include filename="robot_core.xacro" />
-    <xacro:include filename="camera.xacro" />
-    <xacro:include filename="water_tank.xacro" />
-<!-- <xacro:include filename="flexible_rod.xacro" /> -->
+    <!-- <xacro:include filename="camera.xacro" /> -->
     <xacro:include filename="ros2_control.xacro" />
     <xacro:include filename="imu.xacro" />

File: kpi_rover_description/urdf/robot_core.xacro (robot description, xacro)
@@ -2,16 +2,18 @@
 <robot xmlns:xacro="http://www.ros.org/wiki/xacro" >
     <!-- base dimensions -->
-    <xacro:property name="base_x_size" value="0.24" />
-    <xacro:property name="base_y_size" value="0.18" />
-    <xacro:property name="base_z_size" value="0.01" />
+    <xacro:property name="base_x_size" value="0.21" />
+    <xacro:property name="base_y_size" value="0.15" />
+    <xacro:property name="base_z_size" value="0.1" />
     <!-- wheel properties -->
-    <xacro:property name="wheel_length" value="0.04" />
-    <xacro:property name="wheel_radius" value="0.04" />
+    <xacro:property name="wheel_radius" value="$(arg wheel_radius)" />
+    <xacro:property name="axle_separation" value="0.140" />
+    <xacro:property name="wheel_separation" value="0.210" />
+    <xacro:property name="axis_offset_from_base" value="0.035" />
     <!-- material density -->
     <xacro:property name="base_density" value="1500.0" />
     <xacro:property name="wheel_density" value="400.0" />
     <!-- base and wheel mass -->
-    <xacro:property name="base_mass" value="${base_density*base_x_size*base_y_size*base_z_size}" />
-    <xacro:property name="wheel_mass" value="${wheel_density*pi*wheel_radius*wheel_radius*wheel_length}" />
+    <xacro:property name="base_mass" value="2.200" />
+    <xacro:property name="wheel_mass" value="0.035" />
     <!-- base link -->
     <link name="base_link">
@@ -23,18 +25,18 @@
         <parent link="base_footprint"/>
         <child link="base_link"/>
-        <origin xyz="0 0 ${wheel_radius}" rpy="0 0 0"/>
+        <origin xyz="0 0 ${wheel_radius + axis_offset_from_base}" rpy="0 0 0"/>
     </joint>
     <!-- chassis -->
     <link name="chassis">
         <visual>
-        <geometry>
-            <box size="${base_x_size} ${base_y_size} ${base_z_size}"/>
-        </geometry>
-        <material name="white"/>
+            <geometry>
+                <mesh filename = "package://kpi_rover_description/meshes/kpi_rover_body.stl" scale="0.001 0.001 0.001"/>
+            </geometry>
+            <material name="yellow"/>
         </visual>
         <collision>
-        <geometry>
-            <box size="${base_x_size} ${base_y_size} ${base_z_size}"/>
-        </geometry>
+            <geometry>
+                <mesh filename = "package://kpi_rover_description/meshes/kpi_rover_body.stl" scale="0.001 0.001 0.001"/>
+            </geometry>
         </collision>
         <xacro:inertial_box mass="${base_mass}" x="${base_x_size}" y="${base_y_size}" z="${base_z_size}">
@@ -55,5 +57,5 @@
             <visual>
                 <geometry>
-                    <cylinder length="${wheel_length}" radius="${wheel_radius}" />
+                    <cylinder radius="${wheel_radius}" length="-0.027"/>
                 </geometry>
                 <material name="blue"/>
@@ -61,8 +63,8 @@
             <collision>
                 <geometry>
-                    <sphere radius="${wheel_radius}" />
+                    <cylinder radius="${wheel_radius}" length="-0.027"/>
                 </geometry>
             </collision>
-            <xacro:inertial_cylinder mass="${wheel_mass}" length="${wheel_length}" radius="${wheel_radius}">
+            <xacro:inertial_cylinder mass="${wheel_mass}" length="0.020" radius="${wheel_radius}">
                 <origin xyz="0 0 0" rpy="0 0 0"/>
             </xacro:inertial_cylinder>
@@ -71,5 +73,5 @@
             <parent link="base_link"/>
             <child link="${prefix}_link"/>
-            <origin xyz="${x_reflect*(base_x_size/4)} ${y_reflect*(base_y_size + wheel_length)/2} 0" rpy="${-1*y_reflect*pi/2} 0 0"/>
+            <origin xyz="${x_reflect*axle_separation/2} ${y_reflect*wheel_separation/2} ${-axis_offset_from_base}" rpy="${-y_reflect*pi/2} 0 0"/>
             <axis xyz="0 0 ${y_reflect}"/>
         </joint>

File: kpi_rover_description/urdf/ros2_control.xacro (robot description, xacro)
@@ -18,5 +18,5 @@
                 <param name="baud_rate">$(arg baud_rate)</param>
                 <param name="encoder_ticks_per_rev">$(arg encoder_ticks_per_rev)</param>
-                <param name="wheel_radius">0.04</param>
+                <param name="wheel_radius">${wheel_radius}</param>
             </hardware>
             <xacro:wheel_interface prefix="front_left_wheel" />

File: kpi_rover_description/urdf/water_tank.xacro (robot description, xacro)
@@ -1,10 +1,10 @@
 <?xml version="1.0"?>
 <robot xmlns:xacro="http://www.ros.org/wiki/xacro">
-    <xacro:property name="tank_x_size" value="0.15" />
-    <xacro:property name="tank_y_size" value="0.15" />
-    <xacro:property name="tank_z_size" value="0.1" />
-    <xacro:property name="tank_mass" value="1.5" />
-    <xacro:property name="cap_radius" value="0.01" />
-    <xacro:property name="cap_height" value="0.0025" />
+    <xacro:property name="tank_x_size" value="0.6" />
+    <xacro:property name="tank_y_size" value="0.6" />
+    <xacro:property name="tank_z_size" value="0.32" />
+    <xacro:property name="tank_mass" value="100" />
+    <xacro:property name="cap_radius" value="0.1" />
+    <xacro:property name="cap_height" value="0.025" />
     <link name="water_tank_link">
         <visual>

Commit message: Fix IMU position and units

File: kpi_rover_description/urdf/imu.xacro (robot description, xacro)
@@ -4,5 +4,5 @@
         <parent link="base_link"/>
         <child link="imu_link"/>
-        <origin xyz="-0.036 0.039 0.015" rpy="0 0 0"/>
+        <origin xyz="-0.036 0.039 0.015" rpy="0 0 ${pi/2}"/>
     </joint>
     <link name="imu_link"/>
